Commit message: change robot_core wheel

File: AirLab_in_gazebo/description/robot_core.xacro (robot description, xacro)
@@ -85,5 +85,6 @@
         <collision>
             <geometry>
-                <sphere radius="${wheel_radius}"/>
+                <!-- <sphere radius="${wheel_radius}"/> -->
+                <cylinder radius="${wheel_radius}" length="${wheel_thickness}"/>
             </geometry>
         </collision>
@@ -111,5 +112,6 @@
         <collision>
             <geometry>
-                <sphere radius="${wheel_radius}"/>
+                <!-- <sphere radius="${wheel_radius}"/> -->
+                <cylinder radius="${wheel_radius}" length="${wheel_thickness}"/>
             </geometry>
         </collision>
