Commit message: fixed realsense d435i gazebo plugin topic name

File: AirLab_in_gazebo/description/_d435i.gazebo copy.xacro (robot description, xacro)
@@ -159,23 +159,54 @@
             </sensor>
             <!-- IMU -->
-            <sensor name="${camera_name}imu" type="imu">
-                <always_on>true</always_on>
-                <update_rate>${gyro_fps}</update_rate>
-                <!-- <topic>${camera_name}/imu/sample</topic> -->
-                <topic>__default_topic__</topic>
-                <plugin name="${camera_name}imu" filename="libgazebo_ros_imu_sensor.so">
-                      <ros>
-                        <!-- Will publish to /imu/data -->
-                        <namespace>${camera_name}/imu</namespace>
-                        <remapping>~/out:=sample</remapping>
-                    </ros>
-                    <bodyName>${camera_name}_link</bodyName>
-                    <frameName>${gyro_optical_frame}</frameName>
-                    <updateRateHZ>${gyro_fps}</updateRateHZ>
-                    <gaussianNoise>0.1</gaussianNoise>
-                    <xyzOffset>0 0 0</xyzOffset>
-                    <rpyOffset>0 0 0</rpyOffset>
-                </plugin>
-            </sensor>
+            <xacro:if value="${unite_imu_method == 'copy' or unite_imu_method == 'linear_interpolation'}">
+                <sensor name="${camera_name}imu" type="imu">
+                    <always_on>true</always_on>
+                    <update_rate>${gyro_fps}</update_rate>
+                    <topic>${camera_name}/imu/sample</topic>
+                    <plugin name="${camera_name}imu" filename="libgazebo_ros_imu_sensor.so">
+                        <topicName>${camera_name}/imu/sample</topicName>
+                        <bodyName>${camera_name}_link</bodyName>
+                        <frameName>${gyro_optical_frame}</frameName>
+                        <updateRateHZ>${gyro_fps}</updateRateHZ>
+                        <gaussianNoise>0.1</gaussianNoise>
+                        <xyzOffset>0 0 0</xyzOffset>
+                        <rpyOffset>0 0 0</rpyOffset>
+                    </plugin>
+                </sensor>
+            </xacro:if>
+            <!-- Accel and gyro -->
+            <xacro:unless value="${unite_imu_method == 'copy' or unite_imu_method == 'linear_interpolation'}">
+                <sensor name="${camera_name}accel" type="imu">
+                    <always_on>true</always_on>
+                    <update_rate>${accel_fps}</update_rate>
+                    <topic>${camera_name}/accel/sample</topic>
+                    <plugin name="${topics_ns}_accel_plugin" filename="librealsense_gazebo_accel_sensor.so">
+                        <topicName>${camera_name}/accel/sample</topicName>
+                        <bodyName>${camera_name}_link</bodyName>
+                        <updateRateHZ>${accel_fps}</updateRateHZ>
+                        <gaussianNoise>0.1</gaussianNoise>
+                        <xyzOffset>0 0 0</xyzOffset>
+                        <rpyOffset>0 0 0</rpyOffset>
+                        <frameName>${accel_optical_frame}</frameName>
+                        <initialOrientationAsReference>false</initialOrientationAsReference>
+                    </plugin>
+                    <pose>0 0 0 0 0 0</pose>
+                </sensor>
+                <sensor name="${camera_name}gyro" type="imu">
+                    <always_on>true</always_on>
+                    <update_rate>${gyro_fps}</update_rate>
+                    <topic>${camera_name}/gyro/sample</topic>
+                    <plugin name="${topics_ns}_gyro_plugin" filename="librealsense_gazebo_gyro_sensor.so">
+                        <topicName>${camera_name}/gyro/sample</topicName>
+                        <bodyName>${camera_name}_link</bodyName>
+                        <updateRateHZ>${gyro_fps}</updateRateHZ>
+                        <gaussianNoise>0.1</gaussianNoise>
+                        <xyzOffset>0 0 0</xyzOffset>
+                        <rpyOffset>0 0 0</rpyOffset>
+                        <frameName>${gyro_optical_frame}</frameName>
+                        <initialOrientationAsReference>false</initialOrientationAsReference>
+                    </plugin>
+                </sensor>
+            </xacro:unless>
         </gazebo>
         <gazebo>

File: AirLab_in_gazebo/description/_d435i.urdf.xacro (robot description, xacro)
@@ -69,6 +69,6 @@
                 <origin xyz="${d435i_cam_mount_from_center_offset} ${-d435i_cam_depth_py} 0" rpy="${M_PI/2} 0 ${M_PI/2}"/>
                 <geometry>
-                    <!-- <box size="${d435i_cam_width} ${d435i_cam_height} ${d435i_cam_depth}"/> -->
-                    <mesh filename="package://realsense2_description/meshes/d435.dae"/>
+                    <box size="${d435i_cam_width} ${d435i_cam_height} ${d435i_cam_depth}"/>
+                    <!-- <mesh filename="package://realsense2_description/meshes/d435.dae"/> -->
                     <!--<mesh filename="package://realsense2_description/meshes/d435/d435.dae"/>-->
                 </geometry>

File: AirLab_in_gazebo/description/robot.urdf.xacro (robot description, xacro)
@@ -4,4 +4,5 @@
     <xacro:include filename="robot_core.xacro" />
     <xacro:include filename="gazebo_control.xacro" />
+    <!-- <xacro:include filename="imu.xacro" /> -->
     <xacro:include filename="_d435i.urdf.xacro"/>
     <xacro:sensor_d435i parent="chassis" name="D435i_camera" topics_ns="D435i_camera">
