Commit message: add gazebo_control.xacro

File: AirLab_in_gazebo/description/robot.urdf.xacro (robot description, xacro)
@@ -2,4 +2,5 @@
 <robot xmlns:xacro="http://www.ros.org/wiki/xacro"  name="robot">
     <xacro:include filename="robot_core.xacro" />
+    <xacro:include filename="gazebo_control.xacro" />
     <!-- <link name="base_link"></link> -->
     <!-- <xacro:arg name="use_ros2_control" default="true"/>

File: AirLab_in_gazebo/description/robot_core.xacro (robot description, xacro)
@@ -146,5 +146,5 @@
     </link>
     <gazebo reference="caster_wheel">
-        <material>Gazebo/Blcak</material>
+        <material>Gazebo/Black</material>
         <mu1 value="0.001"/>
         <mu2 value="0.001"/>

Commit message: use d435i xacro

File: AirLab_in_gazebo/description/robot.urdf.xacro (robot description, xacro)
@@ -1,7 +1,12 @@
 <?xml version="1.0"?>
 <robot xmlns:xacro="http://www.ros.org/wiki/xacro"  name="robot">
+    <!-- <link name="base_link"></link> -->
     <xacro:include filename="robot_core.xacro" />
     <xacro:include filename="gazebo_control.xacro" />
-    <!-- <link name="base_link"></link> -->
+    <xacro:include filename="_d435i.urdf.xacro"/>
+    <xacro:sensor_d435i parent="chassis" name="D435i_camera" topics_ns="D435i_camera">
+        <origin xyz="-0.01 0.0 0.13" rpy="0.0 0.0 ${pi}"/>
+    </xacro:sensor_d435i>
+    <!-- <xacro:include filename="realsense_d435i.xacro" /> -->
     <!-- <xacro:arg name="use_ros2_control" default="true"/>
     <xacro:arg name="sim_mode" default="false"/>

File: AirLab_in_gazebo/description/robot_core.xacro (robot description, xacro)
@@ -36,5 +36,5 @@
     <!-- BASE_FOOTPRINT LINK -->
     <joint name="base_footprint_joint" type="fixed">
-        <parent link="base_link"/>
+        <parent link="chassis"/>
         <child link="base_footprint"/>
         <origin xyz="0 0 0" rpy="0 0 0"/>

Commit message: test

File: AirLab_in_gazebo/description/robot.urdf.xacro (robot description, xacro)
@@ -1,10 +1,10 @@
 <?xml version="1.0"?>
 <robot xmlns:xacro="http://www.ros.org/wiki/xacro"  name="robot">
-    <!-- <link name="base_link"></link> -->
-    <xacro:include filename="robot_core.xacro" />
-    <xacro:include filename="gazebo_control.xacro" />
+    <link name="base_link"></link>
+    <!-- <xacro:include filename="robot_core.xacro" /> -->
+    <!-- <xacro:include filename="gazebo_control.xacro" /> -->
     <!-- <xacro:include filename="imu.xacro" /> -->
     <xacro:include filename="_d435i.urdf.xacro"/>
-    <xacro:sensor_d435i parent="chassis" name="camera" topics_ns="camera">
+    <xacro:sensor_d435i parent="base_link" name="camera" topics_ns="camera">
         <origin xyz="-0.01 0.0 0.13" rpy="0.0 0.0 ${pi}"/>
     </xacro:sensor_d435i>
