Commit message: 做不出來啦 8-1

File: AirLab_in_gazebo/description/_d435i.gazebo.xacro (robot description, xacro)
@@ -165,5 +165,5 @@
                 <topic>__default_topic__</topic>
                 <plugin name="${camera_name}imu" filename="libgazebo_ros_imu_sensor.so">
-                      <ros>
+                    <ros>
                         <!-- Will publish to /camera/imu -->
                         <!-- <namespace>${camera_name}/imu</namespace> -->

File: AirLab_in_gazebo/description/robot.urdf.xacro (robot description, xacro)
@@ -5,7 +5,11 @@
     <!-- <xacro:include filename="gazebo_control.xacro" /> -->
     <!-- <xacro:include filename="imu.xacro" /> -->
+    <!-- <xacro:include filename="_d435i.urdf.xacro"/>
+    <xacro:sensor_d435i parent="base_link" name="camera" topics_ns="camera">
+        <origin xyz="-0.01 0.0 0.13" rpy="0.0 0.0 ${pi}"/>
+    </xacro:sensor_d435i> -->
     <xacro:include filename="_d435i.urdf.xacro"/>
     <xacro:sensor_d435i parent="base_link" name="camera" topics_ns="camera">
-        <origin xyz="-0.01 0.0 0.13" rpy="0.0 0.0 ${pi}"/>
+        <origin xyz="0.0 0.0 0.13" rpy="0.0 0.0 ${pi}"/>
     </xacro:sensor_d435i>
     <!-- <xacro:include filename="realsense_d435i.xacro" /> -->
