Commit message: trying add depth camera but failed

File: AirLab_in_gazebo/description/gazebo_control.xacro (robot description, xacro)
@@ -4,17 +4,24 @@
         <plugin name="diff_drive" filename="libgazebo_ros_diff_drive.so">
             <!-- Wheel Information -->
-            <left_joint>left_wheel_joint</left_joint>
+            <left_joint>left_wheel_joint</left_joint>       <!-- joint name -->
             <right_joint>right_wheel_joint</right_joint>
-            <wheel_separation>0.297</wheel_separation>
-            <wheel_diameter>0.066</wheel_diameter>
+            <wheel_separation>0.297</wheel_separation>      <!-- the distance from wheel to wheel -->
+            <wheel_diameter>0.06</wheel_diameter>           <!-- wheel diameter -->
             <!-- Limits -->
             <max_wheel_torque>200</max_wheel_torque>
             <max_wheel_acceleration>10.0</max_wheel_acceleration>
             <!-- Output -->
-            <!-- <odometry_frame>odom</odometry_frame>
+            <odometry_frame>odom</odometry_frame>
             <robot_base_frame>base_link</robot_base_frame>
             <publish_odom>true</publish_odom>
             <publish_odom_tf>true</publish_odom_tf>
-            <publish_wheel_tf>true</publish_wheel_tf> -->
+            <publish_wheel_tf>true</publish_wheel_tf>
+            <ros>
+                <!-- Set namespace -->
+                <namespace>/sim</namespace>
+                <!-- Remap default topics -->
+                <remapping>cmd_vel:=cmd_sim</remapping>
+                <remapping>odom:=odom_sim</remapping>
+            </ros>
         </plugin>
     </gazebo>

File: AirLab_in_gazebo/description/robot.urdf.xacro (robot description, xacro)
@@ -1,31 +1,17 @@
 <?xml version="1.0"?>
 <robot xmlns:xacro="http://www.ros.org/wiki/xacro"  name="robot">
-    <!-- <link name="base_link">
-        <origin xyz="0.0 0.0 0.13" rpy="0.0 0.0 0.0"/>
-    </link> -->
-    <xacro:include filename="robot_core.xacro" />
-    <xacro:include filename="gazebo_control.xacro" />
-    <!-- <xacro:include filename="imu.xacro" /> -->
-    <xacro:include filename="_d435i.urdf.xacro"/>
+    <!-- <xacro:include filename="robot_core.xacro" /> -->
+    <!-- <xacro:include filename="gazebo_control.xacro" /> -->
+    <!-- origin is the position between chassis and realsense d435i -->
+    <!-- <xacro:include filename="_d435i.urdf.xacro"/>
     <xacro:sensor_d435i parent="chassis" name="camera" topics_ns="camera">
         <origin xyz="-0.01 0.0 0.13" rpy="0.0 0.0 ${pi}"/>
-    </xacro:sensor_d435i>
+    </xacro:sensor_d435i> -->
+    <!-- Test!! -->
+    <link name="base_link" />
+    <xacro:include filename="depth_camera.xacro" />
     <!-- <xacro:include filename="_d435i.urdf.xacro"/>
     <xacro:sensor_d435i parent="base_link" name="camera" topics_ns="camera">
         <origin xyz="0.0 0.0 0.13" rpy="0.0 0.0 ${pi}"/>
     </xacro:sensor_d435i> -->
-    <!-- <xacro:include filename="realsense_d435i.xacro" /> -->
-    <!-- <xacro:arg name="use_ros2_control" default="true"/>
-    <xacro:arg name="sim_mode" default="false"/>
-    <xacro:include filename="robot_core.xacro" />
-    <xacro:if value="$(arg use_ros2_control)">
-        <xacro:include filename="ros2_control.xacro" />
-    </xacro:if>
-    <xacro:unless value="$(arg use_ros2_control)">
-        <xacro:include filename="gazebo_control.xacro" />
-    </xacro:unless>
-    <xacro:include filename="lidar.xacro" />
-    <xacro:include filename="camera.xacro" /> -->
-    <!-- <xacro:include filename="depth_camera.xacro" /> -->
-    <!-- <xacro:include filename="face.xacro" /> -->
 </robot>

File: AirLab_in_gazebo/description/robot_core.xacro (robot description, xacro)
@@ -67,5 +67,5 @@
     </link>
     <gazebo reference="chassis">
-        <material>Gazebo/White</material>
+        <material>Gazebo/CeilingTiled</material>
     </gazebo>
     <!-- LEFT WHEEL LINK -->
