Commit message: 做不出來啦幹==

File: AirLab_in_gazebo/description/depth_camera.xacro (robot description, xacro)
@@ -1,4 +1,4 @@
 <?xml version="1.0"?>
-<robot xmlns:xacro="http://www.ros.org/wiki/xacro" >
+<robot xmlns:xacro="http://www.ros.org/wiki/xacro">
     <joint name="camera_joint" type="fixed">
         <parent link="base_link"/>
@@ -7,51 +7,33 @@
     </joint>
     <link name="camera_link">
-        <!--  -->
-        <visual>
-            <geometry>
-                <box size="0.010 0.03 0.03"/>
-            </geometry>
-        </visual>
-        <collision>
-            <geometry>
-                <box size="0.010 0.03 0.03"/>
-            </geometry>
-        </collision>
-        <sensor name="camera" type="depth">
-            <always_on>true</always_on>
-            <visualize>true</visualize>
+        <sensor type="depth" name="camera">
+            <always_on>1</always_on>
             <update_rate>30</update_rate>
-            <camera name="intel_realsense_r200">
-                <horizontal_fov>1.02974</horizontal_fov>
-                <image>
-                    <width>640</width>
-                    <height>480</height>
-                    <format>R8G8B8</format>
-                </image>
-                <clip>
-                    <near>0.02</near>
-                    <far>300</far>
-                </clip>
-                <noise>
-                    <type>gaussian</type>
-                    <!-- Noise is sampled independently per pixel on each frame.
-                  That pixel's noise value is added to each of its color
-                  channels, which at that point lie in the range [0,1]. -->
-                    <mean>0.0</mean>
-                    <stddev>0.007</stddev>
-                </noise>
+            <camera name="realsense_r200">
+                <distortion>
+                    <k1>0.1</k1>
+                    <k2>0.2</k2>
+                    <k3>0.3</k3>
+                    <p1>0.4</p1>
+                    <p2>0.5</p2>
+                    <center>0.5 0.5</center>
+                </distortion>
             </camera>
             <plugin name="camera_driver" filename="libgazebo_ros_camera.so">
                 <ros>
-                    <!-- <namespace>test_cam</namespace> -->
-                    <!-- <remapping>image_raw:=image_demo</remapping> -->
-                    <!-- <remapping>camera_info:=camera_info_demo</remapping> -->
+                    <namespace>camera</namespace>
+                    <remapping>camera/image_raw:=camera/custom_image</remapping>
+                    <remapping>camera/image_depth:=camera/custom_image_depth</remapping>
+                    <remapping>camera/camera_info:=camera/custom_info_raw</remapping>
+                    <remapping>camera/camera_info_depth:=camera/custom_info_depth</remapping>
+                    <remapping>camera/points:=camera/custom_points</remapping>
                 </ros>
-                <!-- camera_name>omit so it defaults to sensor name</camera_name-->
-                <!-- frame_name>omit so it defaults to link name</frameName-->
-                <!-- <hack_baseline>0.07</hack_baseline> -->
-                <min_dcamera_driverepth>0.2
-                </min_depth>
-                <max_depth>8.0</max_depth>
+                <!-- Set camera name. If empty, defaults to sensor name (i.e. "sensor_name") -->
+                <!-- <camera_name>sensor_name</camera_name> -->
+                <!-- Set TF frame name. If empty, defaults to link name (i.e. "link_name") -->
+                <!-- <frame_name>camera_link</frame_name> -->
+                <hack_baseline>0.07</hack_baseline>
+                <!-- No need to repeat distortion parameters or to set autoDistortion -->
+                <min_depth>0.001</min_depth>
             </plugin>
         </sensor>

Commit message: change depth camera position

File: AirLab_in_gazebo/description/depth_camera.xacro (robot description, xacro)
@@ -4,5 +4,5 @@
         <parent link="chassis"/>
         <child link="camera_link"/>
-        <origin xyz="0.305 0 0.08" rpy="0 0 0"/>
+        <origin xyz="0.276 0 0.181" rpy="0 0 0"/>
     </joint>
     <link name="camera_link">
@@ -10,4 +10,11 @@
             <geometry>
                 <box size="0.010 0.03 0.03"/>
+            </geometry>
+            <material name="red"/>
+        </visual>
+        <visual>
+            <origin xyz="0 0 -0.05"/>
+            <geometry>
+                <cylinder radius="0.002" length="0.1"/>
             </geometry>
             <material name="red"/>
