Commit message: can read IMU data!

File: AirLab_in_gazebo/description/_d435i.urdf.xacro (robot description, xacro)
@@ -18,5 +18,5 @@
                                           align_depth:=false
                                           enable_pointCloud:=false
-                                          unite_imu_method:=copy
+                                          unite_imu_method:=linear_interpolation
                                           accel_fps:=250
                                           gyro_fps:=400

File: AirLab_in_gazebo/description/robot.urdf.xacro (robot description, xacro)
@@ -4,8 +4,8 @@
     <xacro:include filename="robot_core.xacro" />
     <xacro:include filename="gazebo_control.xacro" />
-    <!-- <xacro:include filename="_d435i.urdf.xacro"/>
+    <xacro:include filename="_d435i.urdf.xacro"/>
     <xacro:sensor_d435i parent="chassis" name="D435i_camera" topics_ns="D435i_camera">
         <origin xyz="-0.01 0.0 0.13" rpy="0.0 0.0 ${pi}"/>
-    </xacro:sensor_d435i> -->
+    </xacro:sensor_d435i>
     <!-- <xacro:include filename="realsense_d435i.xacro" /> -->
     <!-- <xacro:arg name="use_ros2_control" default="true"/>

File: AirLab_in_gazebo/description/robot_core.xacro (robot description, xacro)
@@ -5,8 +5,8 @@
     <xacro:property name="chassis_width" value="0.265"/>
     <xacro:property name="chassis_height" value="0.138"/>
-    <xacro:property name="chassis_mass" value="1.0"/>
+    <xacro:property name="chassis_mass" value="3.0"/>
     <xacro:property name="wheel_radius" value="0.033"/>
     <xacro:property name="wheel_thickness" value="0.026"/>
-    <xacro:property name="wheel_mass" value="0.05"/>
+    <xacro:property name="wheel_mass" value="1"/>
     <xacro:property name="wheel_offset_x" value="0.226"/>
     <xacro:property name="wheel_offset_y" value="0.1485"/>

Commit message: fix d435i xacro file

File: AirLab_in_gazebo/description/_d435i.urdf.xacro (robot description, xacro)
@@ -67,7 +67,9 @@
         <link name="${name}_link">
             <visual>
-                <origin xyz="${d435i_cam_mount_from_center_offset} ${-d435i_cam_depth_py} 0" rpy="${M_PI/2} 0 ${M_PI/2}"/>
+                <!-- <origin xyz="${d435i_cam_mount_from_center_offset} ${-d435i_cam_depth_py} 0" rpy="${M_PI/2} 0 ${M_PI/2}"/> -->
+                <origin xyz="0 ${-d435i_cam_depth_py} 0" rpy="0 0 0"/>
                 <geometry>
-                    <box size="${d435i_cam_width} ${d435i_cam_height} ${d435i_cam_depth}"/>
+                    <box size="${d435i_cam_depth} ${d435i_cam_width} ${d435i_cam_height}"/>
+                    <!-- <box size="${d435i_cam_width} ${d435i_cam_height} ${d435i_cam_depth}"/> -->
                     <!-- <mesh filename="package://realsense2_description/meshes/d435.dae"/> -->
                     <!--<mesh filename="package://realsense2_description/meshes/d435/d435.dae"/>-->

File: AirLab_in_gazebo/description/robot.urdf.xacro (robot description, xacro)
@@ -1,16 +1,18 @@
 <?xml version="1.0"?>
 <robot xmlns:xacro="http://www.ros.org/wiki/xacro"  name="robot">
-    <link name="base_link"></link>
-    <!-- <xacro:include filename="robot_core.xacro" /> -->
-    <!-- <xacro:include filename="gazebo_control.xacro" /> -->
+    <!-- <link name="base_link">
+        <origin xyz="0.0 0.0 0.13" rpy="0.0 0.0 0.0"/>
+    </link> -->
+    <xacro:include filename="robot_core.xacro" />
+    <xacro:include filename="gazebo_control.xacro" />
     <!-- <xacro:include filename="imu.xacro" /> -->
+    <xacro:include filename="_d435i.urdf.xacro"/>
+    <xacro:sensor_d435i parent="chassis" name="camera" topics_ns="camera">
+        <origin xyz="-0.01 0.0 0.13" rpy="0.0 0.0 ${pi}"/>
+    </xacro:sensor_d435i>
     <!-- <xacro:include filename="_d435i.urdf.xacro"/>
     <xacro:sensor_d435i parent="base_link" name="camera" topics_ns="camera">
-        <origin xyz="-0.01 0.0 0.13" rpy="0.0 0.0 ${pi}"/>
+        <origin xyz="0.0 0.0 0.13" rpy="0.0 0.0 ${pi}"/>
     </xacro:sensor_d435i> -->
-    <xacro:include filename="_d435i.urdf.xacro"/>
-    <xacro:sensor_d435i parent="base_link" name="camera" topics_ns="camera">
-        <origin xyz="0.0 0.0 0.13" rpy="0.0 0.0 ${pi}"/>
-    </xacro:sensor_d435i>
     <!-- <xacro:include filename="realsense_d435i.xacro" /> -->
     <!-- <xacro:arg name="use_ros2_control" default="true"/>

Commit message: 修正realsense d435i plugin 圖像大小

File: AirLab_in_gazebo/description/_d435i.urdf.xacro (robot description, xacro)
@@ -12,10 +12,10 @@
     <!--File includes-->
     <xacro:include filename="_d435i.gazebo.xacro"/>
-    <xacro:macro name="sensor_d435i" params="parent
+    <!-- <xacro:macro name="sensor_d435i" params="parent
                                           name:=camera
                                           topics_ns:=camera
-                                          visualize:=false
-                                          align_depth:=false
-                                          enable_pointCloud:=false
+                                          visualize:=true
+                                          align_depth:=true
+                                          enable_pointCloud:=true
                                           unite_imu_method:=linear_interpolation
                                           accel_fps:=250
@@ -25,9 +25,29 @@
                                           depth_height:=720
                                           depth_fps:=30
-                                          infra_width:=640
-                                          infra_height:=480
+                                          infra_width:=1280
+                                          infra_height:=720
                                           infra_fps:=30
                                           color_width:=1920
                                           color_height:=1080
+                                          color_fps:=30
+                                          *origin"> -->
+    <xacro:macro name="sensor_d435i" params="parent
+                                          name:=camera
+                                          topics_ns:=camera
+                                          visualize:=true
+                                          align_depth:=true
+                                          enable_pointCloud:=true
+                                          unite_imu_method:=linear_interpolation
+                                          accel_fps:=63
+                                          gyro_fps:=200
+                                          clip_distance:=-1.0
+                                          depth_width:=848
+                                          depth_height:=480
+                                          depth_fps:=30
+                                          infra_width:=848
+                                          infra_height:=480
+                                          infra_fps:=30
+                                          color_width:=1280
+                                          color_height:=720
                                           color_fps:=30
                                           *origin">

Commit message: 修正小車重量

File: AirLab_in_gazebo/description/_d435i.urdf.xacro (robot description, xacro)
@@ -12,4 +12,5 @@
     <!--File includes-->
     <xacro:include filename="_d435i.gazebo.xacro"/>
+    <!-- 原本的參數 -->
     <!-- <xacro:macro name="sensor_d435i" params="parent
                                           name:=camera
@@ -36,5 +37,5 @@
                                           topics_ns:=camera
                                           visualize:=true
-                                          align_depth:=true
+                                          align_depth:=false
                                           enable_pointCloud:=true
                                           unite_imu_method:=linear_interpolation

File: AirLab_in_gazebo/description/robot.urdf.xacro (robot description, xacro)
@@ -8,5 +8,5 @@
     <xacro:include filename="_d435i.urdf.xacro"/>
     <xacro:sensor_d435i parent="chassis" name="camera" topics_ns="camera">
-        <origin xyz="-0.01 0.0 0.13" rpy="0.0 0.0 ${pi}"/>
+        <origin xyz="0.35 0.0 0.13" rpy="0.0 0.0 0.0"/>
     </xacro:sensor_d435i>
     <!-- Test!! -->

File: AirLab_in_gazebo/description/robot_core.xacro (robot description, xacro)
@@ -5,5 +5,5 @@
     <xacro:property name="chassis_width" value="0.265"/>
     <xacro:property name="chassis_height" value="0.138"/>
-    <xacro:property name="chassis_mass" value="3.0"/>
+    <xacro:property name="chassis_mass" value="5.0"/>
     <xacro:property name="wheel_radius" value="0.033"/>
     <xacro:property name="wheel_thickness" value="0.026"/>
@@ -13,5 +13,5 @@
     <xacro:property name="wheel_offset_z" value="0.01"/>
     <xacro:property name="caster_wheel_radius" value="0.03"/>
-    <xacro:property name="caster_wheel_mass" value="0.01"/>
+    <xacro:property name="caster_wheel_mass" value="3.5"/>
     <xacro:property name="caster_wheel_offset_x" value="0.075"/>
     <xacro:property name="caster_wheel_offset_z" value="${wheel_offset_z - wheel_radius + caster_wheel_radius}"/>

Commit message: test something

File: AirLab_in_gazebo/description/_d435i.urdf.xacro (robot description, xacro)
@@ -102,4 +102,5 @@
                 <geometry>
                     <box size="${d435i_cam_depth} ${d435i_cam_width} ${d435i_cam_height}"/>
+                    <!-- <mesh filename="package://realsense2_description/meshes/d435.dae"/> -->
                 </geometry>
             </collision>

File: AirLab_in_gazebo/description/gazebo_control.xacro (robot description, xacro)
@@ -10,5 +10,5 @@
             <!-- Limits -->
             <max_wheel_torque>200</max_wheel_torque>
-            <max_wheel_acceleration>10.0</max_wheel_acceleration>
+            <max_wheel_acceleration>10</max_wheel_acceleration>
             <!-- Output -->
             <odometry_frame>odom</odometry_frame>

File: AirLab_in_gazebo/description/robot.urdf.xacro (robot description, xacro)
@@ -3,6 +3,4 @@
     <xacro:include filename="robot_core.xacro" />
     <xacro:include filename="gazebo_control.xacro" />
-    <!-- <xacro:include filename="depth_camera.xacro" /> -->
-    <!-- <xacro:include filename="camera.xacro" /> -->
     <!-- origin is the position between chassis and realsense d435i -->
     <xacro:include filename="_d435i.urdf.xacro"/>
@@ -14,7 +12,8 @@
     <!-- <xacro:include filename="depth_camera.xacro" /> -->
     <!-- <xacro:include filename="camera.xacro"/> -->
-    <!-- <xacro:include filename="_d435i.urdf.xacro"/>
+<!--
+    <xacro:include filename="_d435i.urdf.xacro"/>
     <xacro:sensor_d435i parent="base_link" name="camera" topics_ns="camera">
-        <origin xyz="0.0 0.0 0.13" rpy="0.0 0.0 ${pi}"/>
+        <origin xyz="0.0 0.0 0.13" rpy="0.0 0.0 0.0"/>
     </xacro:sensor_d435i> -->
 </robot>
