Commit message: 找到rtab不能用的原因: <ros></ros>

File: AirLab_in_gazebo/description/camera.xacro (robot description, xacro)
@@ -1,23 +1,8 @@
 <?xml version="1.0"?>
 <robot xmlns:xacro="http://www.ros.org/wiki/xacro" >
-    <material name="white">
-        <color rgba="1 1 1 1" />
-    </material>
-    <material name="orange">
-        <color rgba="1 0.3 0.1 1"/>
-    </material>
-    <material name="blue">
-        <color rgba="0.2 0.2 1 1"/>
-    </material>
-    <material name="black">
-        <color rgba="0 0 0 1"/>
-    </material>
-    <material name="red">
-        <color rgba="1 0 0 1"/>
-    </material>
     <joint name="camera_joint" type="fixed">
-        <parent link="base_link"/>
+        <parent link="chassis"/>
         <child link="camera_link"/>
-        <origin xyz="0 0 0.5" rpy="0 0 0"/>
+        <origin xyz="0.276 0 0.181" rpy="0 0.18 0"/>
     </joint>
     <link name="camera_link">
@@ -61,4 +46,5 @@
             </camera>
             <plugin name="camera_controller" filename="libgazebo_ros_camera.so">
+                <frame_name>camera_link_optical</frame_name>
                 <ros>
                     <namespace>custom_ns</namespace>
@@ -66,5 +52,4 @@
                     <remapping>camera_info:=custom_info</remapping>
                 </ros>
-                <frame_name>camera_link_optical</frame_name>
             </plugin>
         </sensor>

File: AirLab_in_gazebo/description/depth_camera.xacro (robot description, xacro)
@@ -1,41 +1,50 @@
 <?xml version="1.0"?>
-<robot xmlns:xacro="http://www.ros.org/wiki/xacro">
+<robot xmlns:xacro="http://www.ros.org/wiki/xacro" >
     <joint name="camera_joint" type="fixed">
-        <parent link="base_link"/>
+        <parent link="chassis"/>
         <child link="camera_link"/>
-        <origin xyz="0 0 1" rpy="0 0 0"/>
+        <origin xyz="0.305 0 0.08" rpy="0 0 0"/>
     </joint>
     <link name="camera_link">
-        <sensor type="depth" name="camera">
-            <always_on>1</always_on>
-            <update_rate>30</update_rate>
-            <camera name="realsense_r200">
-                <distortion>
-                    <k1>0.1</k1>
-                    <k2>0.2</k2>
-                    <k3>0.3</k3>
-                    <p1>0.4</p1>
-                    <p2>0.5</p2>
-                    <center>0.5 0.5</center>
-                </distortion>
+        <visual>
+            <geometry>
+                <box size="0.010 0.03 0.03"/>
+            </geometry>
+            <material name="red"/>
+        </visual>
+    </link>
+    <joint name="camera_optical_joint" type="fixed">
+        <parent link="camera_link"/>
+        <child link="camera_link_optical"/>
+        <origin xyz="0 0 0" rpy="${-pi/2} 0 ${-pi/2}"/>
+    </joint>
+    <link name="camera_link_optical"></link>
+    <gazebo reference="camera_link">
+        <material>Gazebo/Red</material>
+        <sensor name="camera" type="depth">
+            <pose> 0 0 0 0 0 0 </pose>
+            <visualize>true</visualize>
+            <update_rate>10</update_rate>
+            <camera>
+                <horizontal_fov>1.089</horizontal_fov>
+                <image>
+                    <format>B8G8R8</format>
+                    <width>640</width>
+                    <height>480</height>
+                </image>
+                <clip>
+                    <near>0.05</near>
+                    <far>8.0</far>
+                </clip>
             </camera>
-            <plugin name="camera_driver" filename="libgazebo_ros_camera.so">
+            <plugin name="camera_controller" filename="libgazebo_ros_camera.so">
                 <ros>
                     <namespace>camera</namespace>
-                    <remapping>camera/image_raw:=camera/custom_image</remapping>
-                    <remapping>camera/image_depth:=camera/custom_image_depth</remapping>
-                    <remapping>camera/camera_info:=camera/custom_info_raw</remapping>
-                    <remapping>camera/camera_info_depth:=camera/custom_info_depth</remapping>
-                    <remapping>camera/points:=camera/custom_points</remapping>
                 </ros>
-                <!-- Set camera name. If empty, defaults to sensor name (i.e. "sensor_name") -->
-                <!-- <camera_name>sensor_name</camera_name> -->
-                <!-- Set TF frame name. If empty, defaults to link name (i.e. "link_name") -->
-                <!-- <frame_name>camera_link</frame_name> -->
-                <hack_baseline>0.07</hack_baseline>
-                <!-- No need to repeat distortion parameters or to set autoDistortion -->
-                <min_depth>0.001</min_depth>
+                <frame_name>camera_link_optical</frame_name>
+                <min_depth>0.1</min_depth>
+                <max_depth>100.0</max_depth>
             </plugin>
         </sensor>
-    </link>
+    </gazebo>
 </robot>

File: AirLab_in_gazebo/description/gazebo_control.xacro (robot description, xacro)
@@ -17,11 +17,9 @@
             <publish_odom_tf>true</publish_odom_tf>
             <publish_wheel_tf>true</publish_wheel_tf>
-            <ros>
-                <!-- Set namespace -->
+            <!-- <ros>
                 <namespace>/sim</namespace>
-                <!-- Remap default topics -->
                 <remapping>cmd_vel:=cmd_sim</remapping>
                 <remapping>odom:=odom_sim</remapping>
-            </ros>
+            </ros> -->
         </plugin>
     </gazebo>

File: AirLab_in_gazebo/description/robot.urdf.xacro (robot description, xacro)
@@ -1,6 +1,8 @@
 <?xml version="1.0"?>
 <robot xmlns:xacro="http://www.ros.org/wiki/xacro"  name="robot">
-    <!-- <xacro:include filename="robot_core.xacro" /> -->
-    <!-- <xacro:include filename="gazebo_control.xacro" /> -->
+    <xacro:include filename="robot_core.xacro" />
+    <xacro:include filename="gazebo_control.xacro" />
+    <xacro:include filename="depth_camera.xacro" />
+    <!-- <xacro:include filename="camera.xacro" /> -->
     <!-- origin is the position between chassis and realsense d435i -->
     <!-- <xacro:include filename="_d435i.urdf.xacro"/>
@@ -9,7 +11,7 @@
     </xacro:sensor_d435i> -->
     <!-- Test!! -->
-    <link name="base_link" />
+    <!-- <link name="base_link" /> -->
     <!-- <xacro:include filename="depth_camera.xacro" /> -->
-    <xacro:include filename="camera.xacro" />
+    <!-- <xacro:include filename="camera.xacro"/> -->
     <!-- <xacro:include filename="_d435i.urdf.xacro"/>
     <xacro:sensor_d435i parent="base_link" name="camera" topics_ns="camera">

Commit message: try nav2

File: AirLab_in_gazebo/description/camera.xacro (robot description, xacro)
@@ -47,9 +47,4 @@
             <plugin name="camera_controller" filename="libgazebo_ros_camera.so">
                 <frame_name>camera_link_optical</frame_name>
-                <ros>
-                    <namespace>custom_ns</namespace>
-                    <remapping>image_raw:=custom_img</remapping>
-                    <remapping>camera_info:=custom_info</remapping>
-                </ros>
             </plugin>
         </sensor>

File: AirLab_in_gazebo/description/depth_camera.xacro (robot description, xacro)
@@ -4,5 +4,5 @@
         <parent link="chassis"/>
         <child link="camera_link"/>
-        <origin xyz="0.276 0 0.181" rpy="0 0 0"/>
+        <origin xyz="0.305 0 0.08" rpy="0 0 0"/>
     </joint>
     <link name="camera_link">
@@ -10,11 +10,4 @@
             <geometry>
                 <box size="0.010 0.03 0.03"/>
-            </geometry>
-            <material name="red"/>
-        </visual>
-        <visual>
-            <origin xyz="0 0 -0.05"/>
-            <geometry>
-                <cylinder radius="0.002" length="0.1"/>
             </geometry>
             <material name="red"/>
@@ -32,5 +25,5 @@
             <pose> 0 0 0 0 0 0 </pose>
             <visualize>true</visualize>
-            <update_rate>10</update_rate>
+            <update_rate>60</update_rate>
             <camera>
                 <horizontal_fov>1.089</horizontal_fov>
@@ -46,7 +39,4 @@
             </camera>
             <plugin name="camera_controller" filename="libgazebo_ros_camera.so">
-                <ros>
-                    <namespace>camera</namespace>
-                </ros>
                 <frame_name>camera_link_optical</frame_name>
                 <min_depth>0.1</min_depth>

File: AirLab_in_gazebo/description/robot.urdf.xacro (robot description, xacro)
@@ -3,9 +3,10 @@
     <xacro:include filename="robot_core.xacro" />
     <xacro:include filename="gazebo_control.xacro" />
+    <xacro:include filename="depth_camera.xacro" />
     <!-- origin is the position between chassis and realsense d435i -->
-    <xacro:include filename="_d435i.urdf.xacro"/>
+    <!-- <xacro:include filename="_d435i.urdf.xacro"/>
     <xacro:sensor_d435i parent="chassis" name="camera" topics_ns="camera">
         <origin xyz="0.35 0.0 0.13" rpy="0.0 0.0 0.0"/>
-    </xacro:sensor_d435i>
+    </xacro:sensor_d435i> -->
     <!-- Test!! -->
     <!-- <link name="base_link" /> -->
